Commit message: Upgrade my_robot camera into RGBD camera

File: my_robot/urdf/my_robot.xacro (robot description, xacro)
@@ -157,4 +157,11 @@
     <dynamics damping="1.0" friction="1.0"/>
   </joint>
+  <joint name="camera_link_optical" type="fixed">
+    <origin xyz="0 0 0" rpy="-1.5707 0 -1.5707"/>
+    <parent link="camera"/>
+    <child link="camera_link_optical"/>
+  </joint>
+  <link name="camera_link_optical">
+  </link>
   <link name="hokuyo">
     <inertial>
